File: li-ion.sch (KiCad schematic (older format))
At the start: 45 parts, among them J1 18V, J2 AVR-ISP-6, J3 Vout, Q1 4407, Q2 BC847, Q3 4407, Q4 BC847, SW1 SW_Push, SW2 SW_Push, U1 L78L05_SO8, U2 AP1117-33, U3 ATmega8L-8AU, U4 LCD3310, Y1 16MHz

Commit message: Final
Parts:
- removed C15: 10u, symbol Device:CP_Small
- removed C3: 100u, symbol Device:CP_Small
- removed C5: 100n, Capacitor_SMD:C_0805_2012Metric, symbol Device:C_Small
- removed D1, D2: D, symbol Device:D
- removed J3: Vout, symbol Connector_Generic:Conn_01x02
- removed U2: AP1117-33, Package_TO_SOT_SMD:SOT-223-3_TabPin2, symbol Regulator_Linear:AP1117-33
- removed U4: LCD3310, symbol 3310:LCD3310
- added D1, D2: 1N5406, Diode_THT:D_DO-201AD_P15.24mm_Horizontal, symbol Diode:1N5406
- added DS1: WC1602A, Connector_PinHeader_2.54mm:PinHeader_1x16_P2.54mm_Vertical, symbol Display_Character:WC1602A
- added J3, J4, J5, J6: Conn_01x01_Male, Connector_PinHeader_2.54mm:PinHeader_1x01_P2.54mm_Vertical, symbol Connector:Conn_01x01_Male
- added R12: 150, Resistor_SMD:R_0805_2012Metric, symbol Device:R_Small
- added R13, R14: 1R, Resistor_THT:R_Axial_DIN0516_L15.5mm_D5.0mm_P20.32mm_Horizontal, symbol Device:R_Small
- added RV2: 5k, Potentiometer_THT:Potentiometer_Piher_PT-6-V_Vertical, symbol Device:R_POT_Small
- C1: footprint (none) -> Capacitor_THT:C_Radial_D10.0mm_H16.0mm_P5.00mm
- C2: footprint (none) -> Capacitor_THT:C_Radial_D8.0mm_H7.0mm_P3.50mm
- C4: renamed from C6; footprint (none) -> Capacitor_THT:C_Radial_D10.0mm_H16.0mm_P5.00mm
- C5: renamed from C7; footprint Capacitor_SMD:C_0805_2012Metric -> Capacitor_SMD:C_0603_1608Metric
- C7: renamed from C9; footprint (none) -> Capacitor_THT:C_Radial_D10.0mm_H16.0mm_P5.00mm
- C8: renamed from C10; footprint Capacitor_SMD:C_0805_2012Metric -> Capacitor_SMD:C_0603_1608Metric
- J1: footprint (none) -> TerminalBlock_Phoenix:TerminalBlock_Phoenix_MKDS-1,5-2-5.08_1x02_P5.08mm_Horizontal
- L1: value L -> 330uH/2A; footprint (none) -> Inductor_THT:L_Radial_D12.0mm_P5.00mm_Fastron_11P
- L2: value L -> 10u; footprint (none) -> Inductor_SMD:L_6.3x6.3_H3
- R10, R11: footprint Resistor_SMD:R_0805_2012Metric -> Resistor_SMD:R_1206_3216Metric
- RV1: footprint (none) -> Potentiometer_THT:Potentiometer_Piher_PT-6-V_Vertical
- SW1, SW2: footprint (none) -> Button_Switch_THT:SW_Tactile_SPST_Angled_PTS645Vx58-2LFS
- renumbered C12 to C10, C13 to C11, C14 to C12, C4 to C3, C8 to C6, C11 to C9, U3 to U2
Connections:
- net labels added: AVCC, LCD_EN, LCD_RS, LCD_RW
- net labels removed: +3.3V, LCD_CE, LCD_DI, LCD_D_C, LCD_RST, LCD_SCK
- wire segments 166 -> 182
- no-connect marks 10 -> 12
